File: DS100M06V.kicad_pcb (KiCad board)
At the start: 4 copper layers, 81 x 30 mm, 73 parts, among them J2 Wire2Board, J3 wire2board, J4 wire2board, J5 Wire2Board, J6 wire2board, J7 wire2board, SW1 SW_DPDT_x2, U1 AD8039, U2 TEA1-0505, U4 AD8009

Commit message: Offset pot fixed.
Connections:
- RV1 pad 3: -5V -> +5V
Routing:
- net +5V: track 66.1 -> 80.3 mm
Changed lines of the file:
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@@
       (net 9 "Net-(C32-Pad2)") (pinfunction "2") (pintype "passive"))
     (pad "3" thru_hole circle (at -5.08 0 180) (size 1.44 1.44) (drill 0.8) (layers "*.Cu" "*.Mask")
-      (net 7 "-5V") (pinfunction "3") (pintype "passive"))
+      (net 6 "+5V") (pinfunction "3") (pintype "passive"))
     (model "${KICAD6_3DMODEL_DIR}/Potentiometer_THT.3dshapes/Potentiometer_Bourns_3296W_Vertical.wrl"
       (offset (xyz 0 0 0))
@@
   (segment (start 126.3 117.1) (end 130.7 112.7) (width 1) (layer "In2.Cu") (net 6))
   (segment (start 129.6 121.5) (end 127.7 121.5) (width 1) (layer "In2.Cu") (net 6))
+  (segment (start 127.7 121.5) (end 126.3 122.9) (width 1) (layer "In2.Cu") (net 6))
+  (segment (start 126.3 122.9) (end 114.13 122.9) (width 1) (layer "In2.Cu") (net 6))
   (segment (start 157.0125 128.6) (end 157.0125 120.4875) (width 1) (layer "In2.Cu") (net 6))
   (segment (start 157.0125 120.4875) (end 159.2 118.3) (width 1) (layer "In2.Cu") (net 6))
@@
   (segment (start 129.6 119.5) (end 129.6 120.6875) (width 1) (layer "F.Cu") (net 7))
   (segment (start 159.2875 127.4) (end 157.3875 125.5) (width 0.5) (layer "F.Cu") (net 7))
-  (segment (start 109.05 122.05) (end 110.1 121) (width 1) (layer "F.Cu") (net 7))
   (segment (start 128.1 120.6875) (end 128.1125 120.7) (width 0.5) (layer "F.Cu") (net 7))
   (segment (start 128.1125 120.7) (end 130.87 120.7) (width 1) (layer "F.Cu") (net 7))
+  (segment (start 119.3 124.4) (end 125.8 124.4) (width 1) (layer "F.Cu") (net 7))
   (segment (start 151.6 128.6) (end 151.6 127.4125) (width 0.5) (layer "F.Cu") (net 7))
-  (segment (start 114.13 122.9) (end 125.8 122.9) (width 1) (layer "F.Cu") (net 7))
   (segment (start 153.905 124.105) (end 152.025 124.105) (width 0.5) (layer "F.Cu") (net 7))
   (segment (start 129.5 133.1875) (end 129.55 133.1375) (width 0.5) (layer "F.Cu") (net 7))
   (segment (start 159.2875 128.7875) (end 159.3 128.8) (width 0.5) (layer "F.Cu") (net 7))
-  (segment (start 114.13 122.23) (end 114.13 122.9) (width 1) (layer "F.Cu") (net 7))
-  (segment (start 109.05 122.9) (end 109.05 122.05) (width 1) (layer "F.Cu") (net 7))
+  (segment (start 126.9125 120.6875) (end 128.1 120.6875) (width 1) (layer "F.Cu") (net 7))
+  (segment (start 125.8 121.8) (end 126.9125 120.6875) (width 1) (layer "F.Cu") (net 7))
+  (segment (start 115.8 120.9) (end 119.3 124.4) (width 1) (layer "F.Cu") (net 7))
   (segment (start 129.5 134.6) (end 129.5 133.1875) (width 0.5) (layer "F.Cu") (net 7))
-  (segment (start 110.1 121) (end 112.9 121) (width 1) (layer "F.Cu") (net 7))
   (segment (start 128.1 119.5) (end 128.1 120.6875) (width 1) (layer "F.Cu") (net 7))
   (segment (start 155.3 125.5) (end 153.905 124.105) (width 0.5) (layer "F.Cu") (net 7))
-  (segment (start 125.8 122.9) (end 125.8 121.8) (width 1) (layer "F.Cu") (net 7))
   (segment (start 157.3875 125.5) (end 155.3 125.5) (width 0.5) (layer "F.Cu") (net 7))
-  (segment (start 125.8 121.8) (end 126.9125 120.6875) (width 1) (layer "F.Cu") (net 7))
+  (segment (start 109.05 122.9) (end 109.05 122.05) (width 1) (layer "F.Cu") (net 7))
+  (segment (start 109.05 122.05) (end 110.2 120.9) (width 1) (layer "F.Cu") (net 7))
   (segment (start 159.2875 127.35) (end 159.2875 128.7875) (width 1) (layer "F.Cu") (net 7))
   (segment (start 159.2 127.4) (end 159.2875 127.4) (width 0.5) (layer "F.Cu") (net 7))
   (segment (start 151.5875 125.8) (end 151.5875 128.5875) (width 1) (layer "F.Cu") (net 7))
   (segment (start 159.2875 133.4825) (end 159.0125 133.7575) (width 0.5) (layer "F.Cu") (net 7))
+  (segment (start 125.8 124.4) (end 125.8 121.8) (width 1) (layer "F.Cu") (net 7))
   (segment (start 159.2875 128.8125) (end 159.2875 133.4825) (width 1) (layer "F.Cu") (net 7))
   (segment (start 130.87 120.7) (end 131.195 121.025) (width 0.5) (layer "F.Cu") (net 7))
-  (segment (start 126.9125 120.6875) (end 128.1 120.6875) (width 1) (layer "F.Cu") (net 7))
   (segment (start 132.55 112.85) (end 132.55 114.2625) (width 0.5) (layer "F.Cu") (net 7))
   (segment (start 151.5875 128.5875) (end 151.6 128.6) (width 0.5) (layer "F.Cu") (net 7))
-  (segment (start 112.9 121) (end 114.13 122.23) (width 1) (layer "F.Cu") (net 7))
+  (segment (start 110.2 120.9) (end 115.8 120.9) (width 1) (layer "F.Cu") (net 7))
   (segment (start 151.6 127.4125) (end 151.5875 127.4) (width 0.5) (layer "F.Cu") (net 7))
   (segment (start 151.5875 125.8) (end 151.5875 124.5425) (width 1) (layer "F.Cu") (net 7))
   (via (at 129.5 134.6) (size 0.8) (drill 0.4) (layers "F.Cu" "B.Cu") (net 7))
   (via (at 132.55 112.85) (size 0.8) (drill 0.4) (layers "F.Cu" "B.Cu") (net 7))
-  (via (at 125.8 122.9) (size 0.8) (drill 0.4) (layers "F.Cu" "B.Cu") (net 7))
+  (via (at 125.8 124.4) (size 0.8) (drill 0.4) (layers "F.Cu" "B.Cu") (net 7))
   (via (at 151.6 128.6) (size 0.8) (drill 0.4) (layers "F.Cu" "B.Cu") (net 7))
   (via (at 128.1 119.5) (size 0.8) (drill 0.4) (layers "F.Cu" "B.Cu") (net 7))
@@
   (via (at 159.3 128.8) (size 0.8) (drill 0.4) (layers "F.Cu" "B.Cu") (net 7))
   (segment (start 132.55 112.85) (end 132.55 120.85) (width 1) (layer "In2.Cu") (net 7))
+  (segment (start 129.5 128.1) (end 129.5 134.6) (width 1) (layer "In2.Cu") (net 7))
   (segment (start 129.6 119.5) (end 132.55 119.5) (width 1) (layer "In2.Cu") (net 7))
   (segment (start 140.3 128.6) (end 151.6 128.6) (width 1) (layer "In2.Cu") (net 7))
-  (segment (start 125.8 122.9) (end 125.8 124.4) (width 1) (layer "In2.Cu") (net 7))
   (segment (start 132.55 119.5) (end 132.55 112.85) (width 1) (layer "In2.Cu") (net 7))
   (segment (start 125.8 124.4) (end 129.5 128.1) (width 1) (layer "In2.Cu") (net 7))
   (segment (start 132.55 120.85) (end 140.3 128.6) (width 1) (layer "In2.Cu") (net 7))
-  (segment (start 129.5 128.1) (end 129.5 134.6) (width 1) (layer "In2.Cu") (net 7))
   (segment (start 95.45 134.4) (end 97.65 134.4) (width 0.5) (layer "F.Cu") (net 8))
   (segment (start 111.6 126.3875) (end 111.6 122.91) (width 0.5) (layer "F.Cu") (net 9))
@@
         (xy 130.25 112)
         (xy 135 112)
-        (xy 135 112)
-        (xy 143.25 112)
         (xy 143.25 112)
         (xy 157.83 112)
         (xy 157.83 127.5)
         (xy 143.25 127.4)
-        (xy 143.25 127.4)
         (xy 135 127.4)
