File: DS100M06V.kicad_sch (KiCad schematic)
At the start: 73 parts, among them J2 Wire2Board, J3 wire2board, J4 wire2board, J5 Wire2Board, J6 wire2board, J7 wire2board, SW1 SW_DPDT_x2, U1 AD8039, U2 TEA1-0505, U4 AD8009

Commit message: Offset pot fixed.
Connections:
- net +5V: now also RV1.3
- net -5V: no longer RV1.3
Changed lines of the file:
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@@
     )
   )
-  (global_label "-5V" (shape input) (at 158.75 125.73 180) (fields_autoplaced)
+  (global_label "+5V" (shape input) (at 158.75 125.73 180) (fields_autoplaced)
     (effects (font (size 1.27 1.27)) (justify right))
     (property "Intersheetrefs" "${INTERSHEET_REFS}" (at 151.8943 125.73 0)
